Commit message: Add files via upload

File: abi_description/urdf/abi.xacro (robot description, xacro)
@@ -284,4 +284,5 @@
   <axis xyz="0.0 -1.0 0.0"/>
   <limit effort="100" lower="-0.349066" upper="0.174533" velocity="100"/>
+  <dynamics damping="0.1" friction="0.0"/>
 </joint>
 <joint name="l_hip_roll_joint" type="revolute">
@@ -291,4 +292,5 @@
   <axis xyz="0.0 -1.0 0.0"/>
   <limit effort="100" lower="-0.174533" upper="0.349066" velocity="100"/>
+  <dynamics damping="0.1" friction="0.0"/>
 </joint>
 <joint name="r_hip_yaw_joint" type="revolute">
@@ -298,4 +300,5 @@
   <axis xyz="-0.0 -0.0 -1.0"/>
   <limit effort="100" lower="-1.570796" upper="1.570796" velocity="100"/>
+  <dynamics damping="0.1" friction="0.0"/>
 </joint>
 <joint name="l_hip_yaw_joint" type="revolute">
@@ -305,16 +308,21 @@
   <axis xyz="-0.0 -0.0 -1.0"/>
   <limit effort="100" lower="-1.570796" upper="1.570796" velocity="100"/>
-</joint>
-<joint name="l_hip_pitch_joint" type="continuous">
+  <dynamics damping="0.1" friction="0.0"/>
+</joint>
+<joint name="l_hip_pitch_joint" type="revolute">
   <origin rpy="0 0 0" xyz="-0.0235 0.0 -0.024"/>
   <parent link="l_hip_yaw_link_1"/>
   <child link="l_hip_pitch_link__1__1"/>
   <axis xyz="-1.0 -0.0 -0.0"/>
-</joint>
-<joint name="r_hip_pitch_joint" type="continuous">
+  <limit effort="100" lower="-1.570796" upper="1.570796" velocity="100"/>
+  <dynamics damping="0.1" friction="0.0"/>
+</joint>
+<joint name="r_hip_pitch_joint" type="revolute">
   <origin rpy="0 0 0" xyz="-0.0235 0.0 -0.024"/>
   <parent link="r_hip_yaw_link_1"/>
   <child link="r_hip_pitch_link__1__1"/>
   <axis xyz="-1.0 -0.0 -0.0"/>
+  <limit effort="100" lower="-1.570796" upper="1.570796" velocity="100"/>
+  <dynamics damping="0.1" friction="0.0"/>
 </joint>
 <joint name="r_knee_pitch_joint" type="revolute">
@@ -324,4 +332,5 @@
   <axis xyz="-1.0 -0.0 -0.0"/>
   <limit effort="100" lower="-1.919862" upper="0.174533" velocity="100"/>
+  <dynamics damping="0.1" friction="0.0"/>
 </joint>
 <joint name="l_knee_pitch_joint" type="revolute">
@@ -331,4 +340,5 @@
   <axis xyz="1.0 0.0 0.0"/>
   <limit effort="100" lower="-0.174533" upper="1.919862" velocity="100"/>
+  <dynamics damping="0.1" friction="0.0"/>
 </joint>
 <joint name="r_ankle_pitch_joint" type="revolute">
@@ -338,4 +348,5 @@
   <axis xyz="-1.0 -0.0 -0.0"/>
   <limit effort="100" lower="-0.785398" upper="0.785398" velocity="100"/>
+  <dynamics damping="0.1" friction="0.0"/>
 </joint>
 <joint name="l_ankle_pitch_joint" type="revolute">
@@ -345,4 +356,5 @@
   <axis xyz="1.0 -0.0 0.0"/>
   <limit effort="100" lower="-0.785398" upper="0.785398" velocity="100"/>
+  <dynamics damping="0.1" friction="0.0"/>
 </joint>
 <joint name="l_ankle_roll_joint" type="revolute">
@@ -352,4 +364,5 @@
   <axis xyz="-0.0 1.0 -0.0"/>
   <limit effort="100" lower="-0.174533" upper="0.785398" velocity="100"/>
+  <dynamics damping="0.1" friction="0.0"/>
 </joint>
 <joint name="r_ankle_roll_joint" type="revolute">
@@ -359,4 +372,5 @@
   <axis xyz="-0.0 1.0 -0.0"/>
   <limit effort="100" lower="-0.785398" upper="0.174533" velocity="100"/>
+  <dynamics damping="0.1" friction="0.0"/>
 </joint>
 </robot>
